Commit message: Added inertia info for mug.

File: data/mug/mug.urdf (robot description, URDF)
Before this commit: robot mug, 1 links, 0 joints
Links:
- link mug_link: mass None -> 0.1

Commit message: Added obj meshes of mug.

File: data/mug/mug.urdf (robot description, URDF)
Before this commit: robot mug, 1 links, 0 joints
Links:
- link mug_link: geometry collision mesh filename=package://pybullet_sandbox/data/mug/meshes/mug.obj

Commit message: Started working on spawning spheres.

File: data/mug/mug.urdf (robot description, URDF)
Before this commit: robot mug, 1 links, 0 joints
Links:
- link mug_link: geometry collision mesh filename=package://pybullet_sandbox/data/mug/meshes/mug.obj; visual mesh filename=package://pybullet_sandbox/data/mug/meshes/mug.stl
